File: 36keys/name-unneeded.kicad_pcb (KiCad board)
At the start: 2 copper layers, 116 x 105.9 mm, 68 parts, among them SW1 switch, SW10 switch, SW11 switch, SW12 switch, SW13 switch, SW14 switch, SW15 switch, SW16 switch, SW17 switch, SW18 switch, SW19 switch, SW2 switch, SW3 switch, SW4 switch, SW5 switch, SW6 switch, SW7 switch, SW8 switch, SW9 switch, U1 TRRS, U2 ProMicro

Commit message: added pimoroni's footprint.
Parts:
- removed COL1, COL2, COL3, COL4, COL5, F1, F5, F6, F7, GND (x2), RAW, ROW1, ROW2, ROW3, ROW4: Conn_01x01, footprints:wirepad
- removed the D1 at (133.3, 76.2)
- removed the D2 at (133.3, 83.8)
- removed the D3 at (133.3, 86.4)
- removed the D4 at (133.3, 73.7)
- removed G*** (x2): LOGO, footprints:rasu-kulli-khatiah
- removed G*** (x2): LOGO, footprints:hubb-ud-dunya
- removed Ref** (x5): Val**, footprints:hole-m2-pcb
- added H1: MountingHole, footprints:hole-m2-pcb, F.Cu at (39.5, 48.5)
- added H2: MountingHole, footprints:hole-m2-pcb, F.Cu at (39.5, 67.5)
- added H3: MountingHole, footprints:hole-m2-pcb, F.Cu at (96.5, 39.5)
- added H4: MountingHole, footprints:hole-m2-pcb, F.Cu at (96.5, 58.5)
- added H5: MountingHole, footprints:hole-m2-pcb, F.Cu at (113.5, 91.5)
- added J1: Conn_01x05, footprints:pimoroni-trackball-reversible, F.Cu at (118.0, 75.1)
- added R1: R, Resistor_THT:R_Axial_DIN0204_L3.6mm_D1.6mm_P5.08mm_Horizontal, F.Cu at (119.9, 55.9)
- added R2: R, Resistor_THT:R_Axial_DIN0204_L3.6mm_D1.6mm_P5.08mm_Horizontal, F.Cu at (117.6, 55.9)
- moved SW15 8.59 mm to (119.8, 67.1), turned to 90 degrees
- renumbered D17 to D10, D4 to D11, D10 to D12, D15 to D13, D18 to D14, D5 to D15, D11 to D16, D16 to D17, D19 to D18, D7 to D2, D12 to D3, D2 to D4, D8 to D5, D13 to D6, D3 to D7, D9 to D8, D14 to D9, SW17 to SW10, SW4 to SW11, SW9 to SW12, SW15 to SW13, SW18 to SW14, SW11 to SW15, SW5 to SW16, SW10 to SW17, SW16 to SW18, SW6 to SW2, SW12 to SW3, SW2 to SW4, SW7 to SW5, SW13 to SW6, SW3 to SW7, SW14 to SW9, U2 to U1, U1 to U2
Connections:
- SW15 pad 1: Net-(SW11-Pad1) -> VCC
- SW15 pad 2: Net-(SW11-Pad2) -> GND
- U1 pad 1: Net-(PD3-Pad1) -> (no net)
- U1 pad 17: Net-(PF7-Pad1) -> (no net)
- U1 pad 18: Net-(PF6-Pad1) -> (no net)
- U1 pad 19: Net-(PF5-Pad1) -> (no net)
- U1 pad 2: Net-(PD2-Pad1) -> DATA
- U1 pad 20: Net-(PF1-Pad1) -> (no net)
- U1 pad 21: Net-(U1-Pad2) -> VCC
- U1 pad 22: Net-(SW11-Pad1) -> (no net)
- U1 pad 23: Net-(SW11-Pad2) -> GND
- U1 pad 24: Net-(RAW1-Pad1) -> (no net)
- U1 pad 3: Net-(GND1-Pad1) -> GND
- U1 pad 4: Net-(GND2-Pad1) -> GND
- U1 pad 5: Net-(PD1-Pad1) -> SCL
- U1 pad 7: Net-(PD4-Pad1) -> (no net)
- U2 pad 1: SDA -> DATA
- U2 pad 2: Net-(U1-Pad2) -> VCC
- U2 pad 3: Net-(SW11-Pad2) -> (no net)
- U2 pad 4: Net-(U1-Pad4) -> GND
Routing:
- net GND: track 0.00 -> 106.0 mm
- net COL2: track 307.5 -> 208.8 mm
- net COL0: track 307.3 -> 217.1 mm
- net Net-(SW11-Pad2): track 89.9 -> 0.00 mm
- net Net-(RAW1-Pad1): track 88.1 -> 0.00 mm
- net Net-(SW11-Pad1): track 83.1 -> 0.00 mm
- net COL1: track 271.8 -> 191.1 mm
- net Net-(PD3-Pad1): track 77.8 -> 0.00 mm
- net VCC: track 0.00 -> 75.5 mm
- net Net-(PD2-Pad1): track 72.3 -> 0.00 mm
- net SCL: track 0.00 -> 68.5 mm
- net Net-(GND1-Pad1): track 66.9 -> 0.00 mm
- net Net-(PF1-Pad1): track 65.1 -> 0.00 mm
- net Net-(PF5-Pad1): track 65.0 -> 0.00 mm
- net Net-(PF7-Pad1): track 65.0 -> 0.00 mm
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Other:
- outline, holes or cut-outs redrawn
