File: 36keys/name-unneeded.sch (KiCad schematic (older format))
At the start: 59 parts, among them SW1 switch, SW10 switch, SW11 switch, SW12 switch, SW13 switch, SW14 switch, SW15 switch, SW16 switch, SW17 switch, SW18 switch, SW19 switch, SW2 switch, SW3 switch, SW4 switch, SW5 switch, SW6 switch, SW7 switch, SW8 switch, SW9 switch, U1 TRRS, U2 ProMicro

Commit message: added pimoroni's footprint.
Parts:
- removed GND1, GND2, PD1, PD2, PD3, PD4, PF1, PF5, PF6, PF7, RAW1, XCOL1, XCOL2, XCOL3, XCOL4, XCOL5, XROW1, XROW2, XROW3, XROW4: Conn_01x01, footprints:wirepad, symbol Connector_Generic:Conn_01x01
- added H1, H2, H3, H4, H5: MountingHole, footprints:hole-m2-pcb, symbol mechanical:MountingHole
- added J1: Conn_01x05, footprints:pimoroni-trackball-reversible, symbol Connector_Generic:Conn_01x05
- added R1, R2: R, Resistor_THT:R_Axial_DIN0204_L3.6mm_D1.6mm_P5.08mm_Horizontal, symbol Device:R
- renumbered D17 to D10, D4 to D11, D10 to D12, D15 to D13, D18 to D14, D5 to D15, D11 to D16, D16 to D17, D19 to D18, D7 to D2, D12 to D3, D2 to D4, D8 to D5, D13 to D6, D3 to D7, D9 to D8, D14 to D9, SW17 to SW10, SW4 to SW11, SW9 to SW12, SW15 to SW13, SW18 to SW14, SW11 to SW15, SW5 to SW16, SW10 to SW17, SW16 to SW18, SW6 to SW2, SW12 to SW3, SW2 to SW4, SW7 to SW5, SW13 to SW6, SW3 to SW7, SW14 to SW9, U2 to U1, U1 to U2
Connections:
- net labels added: DATA, GND, SCL, VCC
- wire segments 71 -> 54
- no-connect marks 1 -> 0
Other:
- moved on the sheet: SW15, U1, U2
